File: Diff Simulator/Diff Simulator.sch (KiCad schematic (older format))
At the start: 9 parts

Commit message: Mitch updated diff amp sim files
Parts:
- removed U?: AD8276, symbol Amplifier_Difference:AD8276
- removed V2: 0.55, symbol pspice:VSOURCE
- added U1: AD8276, symbol Amplifier_Difference:AD8276
- R1, R2: Spice_Model 1000 -> (none); Spice_Netlist_Enabled Y -> (none); Spice_Primitive R -> (none)
- R3, R4: value 5400 -> 2000; Spice_Model 5400 -> 2000
- V1: Spice_Model dc 1.65 ac 1.1 sin(1.65 1.1 1k) -> sin(0 1 2k)
Connections:
- net VCC: now also U1.7 (V+)
- net VEE: now also U1.4 (V-)
- net Vout: now also U1.6
- net at R3.2: now also R1.1, U1.2 (-); no longer R2.1
- net GND: now reaches R4.2
- net GND: now also R1.2, V1.2 (E2), V3.2 (E2), V4.2 (E2); no longer R1.1
- removed net 0: R1.2, R4.1, V1.2 (E2), V3.2 (E2), V4.2 (E2)
- new net: R2.1, R4.1, U1.3 (+)
- no-connect marks 2 -> 0
Other:
- moved on the sheet: R3, R4
Changed lines of the file:
@@
 EESchema Schematic File Version 4
+LIBS:Diff Simulator-cache
 EELAYER 30 0
 EELAYER END
@@
 $EndDescr
 $Comp
+L power:GND #PWR0105
+U 1 1 5F715225
+P 4700 4350
+F 0 "#PWR0105" H 4700 4100 50  0001 C CNN
+F 1 "GND" H 4705 4177 50  0000 C CNN
+F 2 "" H 4700 4350 50  0001 C CNN
+F 3 "" H 4700 4350 50  0001 C CNN
+F 4 "I" H 4700 4350 50  0001 C CNN "Spice_Primitive"
+F 5 "dc 0" H 4700 4350 50  0001 C CNN "Spice_Model"
+F 6 "Y" H 4700 4350 50  0001 C CNN "Spice_Netlist_Enabled"
+	1    4700 4350
+	1    0    0    -1
+$EndComp
+$Comp
 L Device:R R3
 U 1 1 5F716D8C
-P 5100 4050
-F 0 "R3" V 4893 4050 50  0000 C CNN
-F 1 "5400" V 4984 4050 50  0000 C CNN
-F 2 "" V 5030 4050 50  0001 C CNN
-F 3 "~" H 5100 4050 50  0001 C CNN
-F 4 "R" H 5100 4050 50  0001 C CNN "Spice_Primitive"
-F 5 "5400" H 5100 4050 50  0001 C CNN "Spice_Model"
-F 6 "Y" H 5100 4050 50  0001 C CNN "Spice_Netlist_Enabled"
-	1    5100 4050
+P 5100 2750
+F 0 "R3" V 4893 2750 50  0000 C CNN
+F 1 "2000" V 4984 2750 50  0000 C CNN
+F 2 "" V 5030 2750 50  0001 C CNN
+F 3 "~" H 5100 2750 50  0001 C CNN
+F 4 "R" H 5100 2750 50  0001 C CNN "Spice_Primitive"
+F 5 "2000" H 5100 2750 50  0001 C CNN "Spice_Model"
+F 6 "Y" H 5100 2750 50  0001 C CNN "Spice_Netlist_Enabled"
+	1    5100 2750
 	0    1    1    0
 $EndComp
@@
 F 2 "" V 4430 3600 50  0001 C CNN
 F 3 "~" H 4500 3600 50  0001 C CNN
-F 4 "R" H 4500 3600 50  0001 C CNN "Spice_Primitive"
-F 5 "1000" H 4500 3600 50  0001 C CNN "Spice_Model"
-F 6 "Y" H 4500 3600 50  0001 C CNN "Spice_Netlist_Enabled"
 	1    4500 3600
 	0    1    1    0
@@
 F 2 "" V 4480 3100 50  0001 C CNN
 F 3 "~" H 4550 3100 50  0001 C CNN
-F 4 "R" H 4550 3100 50  0001 C CNN "Spice_Primitive"
-F 5 "1000" H 4550 3100 50  0001 C CNN "Spice_Model"
-F 6 "Y" H 4550 3100 50  0001 C CNN "Spice_Netlist_Enabled"
 	1    4550 3100
 	0    1    1    0
@@
 L Device:R R4
 U 1 1 5F717E7F
-P 4850 2800
-F 0 "R4" H 4920 2846 50  0000 L CNN
-F 1 "5400" H 4920 2755 50  0000 L CNN
-F 2 "" V 4780 2800 50  0001 C CNN
-F 3 "~" H 4850 2800 50  0001 C CNN
-F 4 "R" H 4850 2800 50  0001 C CNN "Spice_Primitive"
-F 5 "5400" H 4850 2800 50  0001 C CNN "Spice_Model"
-F 6 "Y" H 4850 2800 50  0001 C CNN "Spice_Netlist_Enabled"
-	1    4850 2800
+P 4700 4150
+F 0 "R4" H 4770 4196 50  0000 L CNN
+F 1 "2000" H 4770 4105 50  0000 L CNN
+F 2 "" V 4630 4150 50  0001 C CNN
+F 3 "~" H 4700 4150 50  0001 C CNN
+F 4 "R" H 4700 4150 50  0001 C CNN "Spice_Primitive"
+F 5 "2000" H 4700 4150 50  0001 C CNN "Spice_Model"
+F 6 "Y" H 4700 4150 50  0001 C CNN "Spice_Netlist_Enabled"
+	1    4700 4150
 	1    0    0    -1
 $EndComp
@@
 	4100 3600 4350 3600
 Wire Wire Line
-	4700 3100 4850 3100
+	4700 3100 4900 3100
 Wire Wire Line
 	4900 3350 4950 3350
@@
 Vout
 $Comp
-L pspice:VSOURCE V2
-U 1 1 5F728989
-P 2700 1600
-F 0 "V2" H 2928 1646 50  0000 L CNN
-F 1 "0.55" H 2928 1555 50  0000 L CNN
-F 2 "" H 2700 1600 50  0001 C CNN
-F 3 "~" H 2700 1600 50  0001 C CNN
-F 4 "V" H 2700 1600 50  0001 C CNN "Spice_Primitive"
-F 5 "dc 550m" H 2700 1600 50  0001 C CNN "Spice_Model"
-F 6 "Y" H 2700 1600 50  0001 C CNN "Spice_Netlist_Enabled"
-	1    2700 1600
+L pspice:VSOURCE V3
+U 1 1 5F726361
+P 1850 1600
+F 0 "V3" H 2078 1646 50  0000 L CNN
+F 1 "13" H 2078 1555 50  0000 L CNN
+F 2 "" H 1850 1600 50  0001 C CNN
+F 3 "~" H 1850 1600 50  0001 C CNN
+F 4 "V" H 1850 1600 50  0001 C CNN "Spice_Primitive"
+F 5 "dc 13" H 1850 1600 50  0001 C CNN "Spice_Model"
+F 6 "Y" H 1850 1600 50  0001 C CNN "Spice_Netlist_Enabled"
+	1    1850 1600
+	1    0    0    -1
+$EndComp
+Wire Wire Line
+	1850 1300 1850 1100
+Wire Wire Line
+	1850 2100 1850 1900
+Text GLabel 1850 1100 1    50   Input ~ 0
+VCC
+Text GLabel 5150 3750 3    50   Input ~ 0
+VCC
+$Comp
+L power:GND #PWR02
+U 1 1 5F727D6E
+P 1850 2100
+F 0 "#PWR02" H 1850 1850 50  0001 C CNN
+F 1 "GND" H 1855 1927 50  0000 C CNN
+F 2 "" H 1850 2100 50  0001 C CNN
+F 3 "" H 1850 2100 50  0001 C CNN
+	1    1850 2100
 	1    0    0    -1
 $EndComp
@@
 F 3 "~" H 3700 1600 50  0001 C CNN
 F 4 "V" H 3700 1600 50  0001 C CNN "Spice_Primitive"
-F 5 "dc 1.65 ac 1.1 sin(1.65 1.1 1k)" H 3700 1600 50  0001 C CNN "Spice_Model"
+F 5 "sin(0 1 2k)" H 3700 1600 50  0001 C CNN "Spice_Model"
 F 6 "Y" H 3700 1600 50  0001 C CNN "Spice_Netlist_Enabled"
 	1    3700 1600
@@
 $EndComp
 Wire Wire Line
-	2700 1300 2700 1050
-Wire Wire Line
 	3700 1000 3700 1300
 Wire Wire Line
 	3700 1900 3700 2300
-Wire Wire Line
-	2700 2250 2700 1900
+$Comp
+L power:GND #PWR04
+U 1 1 5F72A626
+P 3700 2300
+F 0 "#PWR04" H 3700 2050 50  0001 C CNN
+F 1 "GND" H 3705 2127 50  0000 C CNN
+F 2 "" H 3700 2300 50  0001 C CNN
+F 3 "" H 3700 2300 50  0001 C CNN
+	1    3700 2300
+	1    0    0    -1
+$EndComp
 Text GLabel 3700 1000 1    50   Input ~ 0
 V1
-Text GLabel 2700 1050 1    50   Input ~ 0
-V2
 Text Notes 5650 2200 2    50   ~ 0
 .tran 1u 1m
-Wire Wire Line
-	4900 3350 4900 3100
-Wire Wire Line
-	5250 4050 5750 4050
-Wire Wire Line
-	4950 3600 4950 3550
-Wire Wire Line
-	4650 3600 4850 3600
-Wire Wire Line
-	5550 3450 5750 3450
-Wire Wire Line
-	4850 2450 4850 2650
-Wire Wire Line
-	4850 2950 4850 3100
-Connection ~ 4850 3100
-Wire Wire Line
-	4850 3100 4900 3100
-Wire Wire Line
-	4850 3600 4850 4050
-Connection ~ 4850 3600
-Wire Wire Line
-	4850 3600 4950 3600
-Wire Wire Line
-	5750 4050 5750 3450
-Connection ~ 5750 3450
-Wire Wire Line
-	5750 3450 5950 3450
-Wire Wire Line
-	4850 4050 4950 4050
-$Comp
-L pspice:VSOURCE V3
-U 1 1 5F827CA6
-P 1850 1500
-F 0 "V3" H 2078 1546 50  0000 L CNN
-F 1 "13" H 2078 1455 50  0000 L CNN
-F 2 "" H 1850 1500 50  0001 C CNN
-F 3 "~" H 1850 1500 50  0001 C CNN
-F 4 "V" H 1850 1500 50  0001 C CNN "Spice_Primitive"
-F 5 "dc 13" H 1850 1500 50  0001 C CNN "Spice_Model"
-F 6 "Y" H 1850 1500 50  0001 C CNN "Spice_Netlist_Enabled"
-	1    1850 1500
-	1    0    0    -1
-$EndComp
-$Comp
-L pspice:VSOURCE V4
-U 1 1 5F8282BF
-P 1100 1550
-F 0 "V4" H 1328 1596 50  0000 L CNN
-F 1 "-13" H 1328 1505 50  0000 L CNN
-F 2 "" H 1100 1550 50  0001 C CNN
-F 3 "~" H 1100 1550 50  0001 C CNN
-F 4 "V" H 1100 1550 50  0001 C CNN "Spice_Primitive"
-F 5 "dc -13" H 1100 1550 50  0001 C CNN "Spice_Model"
-F 6 "Y" H 1100 1550 50  0001 C CNN "Spice_Netlist_Enabled"
-	1    1100 1550
-	1    0    0    -1
-$EndComp
-Text GLabel 1850 900  1    50   Input ~ 0
-VCC
-Text GLabel 1100 1050 1    50   Input ~ 0
-VEE
-Wire Wire Line
-	1850 1950 1850 1800
-Wire Wire Line
-	1850 1200 1850 900
-Wire Wire Line
-	1100 1050 1100 1250
-Wire Wire Line
-	1100 1850 1100 2000
-Text GLabel 1100 2000 3    50   Input ~ 0
-GND
-Text GLabel 1850 1950 3    50   Input ~ 0
-GND
-Text GLabel 2700 2250 3    50   Input ~ 0
-GND
-Text GLabel 3700 2300 3    50   Input ~ 0
-GND
-$Comp
-L pspice:0 #GND?
-U 1 1 5F82E284
-P 2100 3600
-F 0 "#GND?" H 2100 3500 50  0001 C CNN
-F 1 "0" H 2100 3689 50  0000 C CNN
-F 2 "" H 2100 3600 50  0001 C CNN
-F 3 "~" H 2100 3600 50  0001 C CNN
-F 4 "I" H 2100 3600 50  0001 C CNN "Spice_Primitive"
-F 5 "dc 0" H 2100 3600 50  0001 C CNN "Spice_Model"
-F 6 "Y" H 2100 3600 50  0001 C CNN "Spice_Netlist_Enabled"
-	1    2100 3600
-	1    0    0    -1
-$EndComp
-Text GLabel 2100 3550 1    50   Input ~ 0
-GND
-Wire Wire Line
-	2100 3550 2100 3600
-NoConn ~ 5250 3150
 Text GLabel 5150 3150 1    50   Input ~ 0
 VEE
-Text GLabel 5150 3750 3    50   Input ~ 0
-VCC
-$Comp
-L power:GND #PWR?
-U 1 1 5F83F1B4
+$Comp
+L pspice:VSOURCE V4
+U 1 1 5F72E756
+P 1000 1650
+F 0 "V4" H 1228 1696 50  0000 L CNN
+F 1 "-13" H 1228 1605 50  0000 L CNN
+F 2 "" H 1000 1650 50  0001 C CNN
+F 3 "~" H 1000 1650 50  0001 C CNN
+F 4 "V" H 1000 1650 50  0001 C CNN "Spice_Primitive"
+F 5 "dc -13" H 1000 1650 50  0001 C CNN "Spice_Model"
+F 6 "Y" H 1000 1650 50  0001 C CNN "Spice_Netlist_Enabled"
+	1    1000 1650
+	1    0    0    -1
+$EndComp
+Text GLabel 1000 1350 1    50   Input ~ 0
+VEE
+$Comp
+L power:GND #PWR01
+U 1 1 5F72F2E6
+P 1000 1950
+F 0 "#PWR01" H 1000 1700 50  0001 C CNN
+F 1 "GND" H 1005 1777 50  0000 C CNN
+F 2 "" H 1000 1950 50  0001 C CNN
+F 3 "" H 1000 1950 50  0001 C CNN
+	1    1000 1950
+	1    0    0    -1
+$EndComp
+Wire Wire Line
+	4900 3350 4900 3100
+Wire Wire Line
+	4900 3100 4900 2750
+Wire Wire Line
+	4900 2750 4950 2750
+Connection ~ 4900 3100
+Wire Wire Line
+	5250 2750 5750 2750
+Wire Wire Line
+	5750 2750 5750 3450
+Connection ~ 5750 3450
+Wire Wire Line
+	5750 3450 5950 3450
+Wire Wire Line
+	4700 4300 4700 4350
+Wire Wire Line
+	4650 3600 4700 3600
+Wire Wire Line
+	4950 3600 4950 3550
+Wire Wire Line
+	4700 3600 4700 4000
+Connection ~ 4700 3600
+Wire Wire Line
+	4700 3600 4950 3600
+$Comp
+L power:GND #PWR03
+U 1 1 5F826BC0
 P 4100 3100
-F 0 "#PWR?" H 4100 2850 50  0001 C CNN
+F 0 "#PWR03" H 4100 2850 50  0001 C CNN
 F 1 "GND" H 4105 2927 50  0000 C CNN
 F 2 "" H 4100 3100 50  0001 C CNN
@@
 	1    0    0    -1
 $EndComp
-$Comp
-L power:GND #PWR?
-U 1 1 5F83F58A
-P 4850 2450
-F 0 "#PWR?" H 4850 2200 50  0001 C CNN
-F 1 "GND" H 4855 2277 50  0000 C CNN
-F 2 "" H 4850 2450 50  0001 C CNN
-F 3 "" H 4850 2450 50  0001 C CNN
-	1    4850 2450
-	1    0    0    -1
-$EndComp
-$Comp
-L Amplifier_Difference:AD8276 U?
-U 1 1 5F8400B7
+Wire Wire Line
+	5550 3450 5750 3450
+$Comp
+L Amplifier_Difference:AD8276 U1
+U 1 1 5F82850A
 P 5250 3450
-F 0 "U?" H 5594 3404 50  0000 L CNN
+F 0 "U1" H 5594 3404 50  0000 L CNN
 F 1 "AD8276" H 5594 3495 50  0000 L CNN
 F 2 "" H 5250 3450 50  0001 C CNN
@@
 F 5 "AD8276" H 5250 3450 50  0001 C CNN "Spice_Model"
 F 6 "Y" H 5250 3450 50  0001 C CNN "Spice_Netlist_Enabled"
-F 7 "3 2 7 4 6 1 5" H 5250 3450 50  0001 C CNN "Spice_Node_Sequence"
-F 8 "ad8276.cir" H 5250 3450 50  0001 C CNN "Spice_Lib_File"
+F 7 "ad8276.cir" H 5250 3450 50  0001 C CNN "Spice_Lib_File"
+F 8 "3 2 7 4 6 1 5" H 5250 3450 50  0001 C CNN "Spice_Node_Sequence"
 	1    5250 3450
 	1    0    0    1
 $EndComp
-NoConn ~ 5250 3750
 $EndSCHEMATC
