File: LAUNCHXL-F28379D_Breakout.sch (KiCad schematic (older format))
At the start: 20 parts, among them IC1 LM358N, Q1 100V/17A, Q2 100V/17A, Q3 100V/17A, Q4 100V/17A, Q5 100V/17A, Q6 100V/17A

Commit message: LTSpice Simulation Finished
Parts:
- removed C1: 0.1uF, Capacitor_SMD:C_0805_2012Metric_Pad1.15x1.40mm_HandSolder, symbol Device:C
- removed IC1: LM358N, Package_DIP:DIP-8_W7.62mm_Socket, symbol PCB_2020:LM358N
- removed R3: 3k, Resistor_SMD:R_0805_2012Metric_Pad1.15x1.40mm_HandSolder, symbol Device:R
- removed R4: 6.8k, Resistor_SMD:R_0805_2012Metric_Pad1.15x1.40mm_HandSolder, symbol Device:R
- added R3, R4: 1000, symbol PCB_2020-rescue:R-Device
- added R6, R7: 5400, symbol PCB_2020-rescue:R-Device
- added U2: TL084CN, symbol PCB_2020:TL084CN
- CONN2: symbol Connector:Conn_01x08_Male -> PCB_2020-rescue:Conn_01x08_Male-Connector
- CONN5: symbol Connector:Conn_01x04_Male -> PCB_2020-rescue:Conn_01x04_Male-Connector
- CONN6: symbol Connector:Conn_01x06_Male -> PCB_2020-rescue:Conn_01x06_Male-Connector
- CONN7, DCDC_CONN_12V: symbol Connector:Conn_01x02_Male -> PCB_2020-rescue:Conn_01x02_Male-Connector
- JETSON_CONN_PWR: symbol Connector:Conn_01x03_Male -> PCB_2020-rescue:Conn_01x03_Male-Connector
- Q1, Q2, Q3, Q4, Q5, Q6: symbol Device:Q_NMOS_GDS -> PCB_2020-rescue:Q_NMOS_GDS-Device
- R1, R18, R2, R5: symbol Device:R -> PCB_2020-rescue:R-Device
Connections:
- net labels added: +12V-power, +3V3-power, +5V-power, GND-power
- net labels removed: +12V, +3V3, +5V, GND

Commit message: updated pcb
Parts:
- R3, R4, R6, R7: footprint (none) -> Resistor_SMD:R_0805_2012Metric_Pad1.15x1.40mm_HandSolder
- U2: footprint (none) -> Drivetrain_control:TL084CN
Changed lines of the file:
@@
 F 0 "U2" H 4544 3896 50  0000 L CNN
 F 1 "TL084CN" H 4544 3805 50  0000 L CNN
-F 2 "" H 4400 3600 50  0001 C CNN
+F 2 "Drivetrain_control:TL084CN" H 4400 3600 50  0001 C CNN
 F 3 "" H 4400 3600 50  0001 C CNN
 	1    4100 3850
@@
 F 0 "R3" V 3143 3950 50  0000 C CNN
 F 1 "1000" V 3234 3950 50  0000 C CNN
-F 2 "" V 3280 3950 50  0001 C CNN
+F 2 "Resistor_SMD:R_0805_2012Metric_Pad1.15x1.40mm_HandSolder" V 3280 3950 50  0001 C CNN
 F 3 "" H 3350 3950 50  0001 C CNN
 	1    3350 3950
@@
 F 0 "R7" V 4093 4750 50  0000 C CNN
 F 1 "5400" V 4184 4750 50  0000 C CNN
-F 2 "" V 4230 4750 50  0001 C CNN
+F 2 "Resistor_SMD:R_0805_2012Metric_Pad1.15x1.40mm_HandSolder" V 4230 4750 50  0001 C CNN
 F 3 "" H 4300 4750 50  0001 C CNN
 	1    4300 4750
@@
 F 0 "R6" H 3420 3096 50  0000 L CNN
 F 1 "5400" H 3420 3005 50  0000 L CNN
-F 2 "" V 3280 3050 50  0001 C CNN
+F 2 "Resistor_SMD:R_0805_2012Metric_Pad1.15x1.40mm_HandSolder" V 3280 3050 50  0001 C CNN
 F 3 "" H 3350 3050 50  0001 C CNN
 	1    3350 3050
@@
 F 0 "R4" V 2893 3400 50  0000 C CNN
 F 1 "1000" V 2984 3400 50  0000 C CNN
-F 2 "" V 3030 3400 50  0001 C CNN
+F 2 "Resistor_SMD:R_0805_2012Metric_Pad1.15x1.40mm_HandSolder" V 3030 3400 50  0001 C CNN
 F 3 "" H 3100 3400 50  0001 C CNN
 	1    3100 3400

Commit message: Updating PCB
Parts:
- added C1, C3: 0.022uF, Capacitor_SMD:C_0805_2012Metric_Pad1.18x1.45mm_HandSolder, symbol PCB_2020-rescue:C-Device
- added R8: 5000, Resistor_SMD:R_0612_1632Metric_Pad1.18x3.40mm_HandSolder, symbol PCB_2020-rescue:R-Device
- added R9: 1000, Resistor_SMD:R_0612_1632Metric_Pad1.18x3.40mm_HandSolder, symbol PCB_2020-rescue:R-Device
- added U3: DRV8874, Drivetrain_control:DRV8874PWPR, symbol PCB_2020:DRV8874
- R1, R18, R2, R3, R4, R5, R6, R7: footprint Resistor_SMD:R_0805_2012Metric_Pad1.15x1.40mm_HandSolder -> Resistor_SMD:R_0612_1632Metric_Pad1.18x3.40mm_HandSolder
Connections:
- wire segments 70 -> 89
- no-connect marks 0 -> 1
Changed lines of the file:
@@
 F 0 "R1" H 4600 1550 59  0000 L BNN
 F 1 "10k" H 4550 1450 59  0000 L BNN
-F 2 "Resistor_SMD:R_0805_2012Metric_Pad1.15x1.40mm_HandSolder" H 4800 1500 50  0001 C CNN
+F 2 "Resistor_SMD:R_0612_1632Metric_Pad1.18x3.40mm_HandSolder" H 4800 1500 50  0001 C CNN
 F 3 "" H 4800 1500 50  0001 C CNN
 	1    4800 1500
@@
 F 0 "R5" H 6550 2759 59  0000 L BNN
 F 1 "560" H 6550 2570 59  0000 L BNN
-F 2 "Resistor_SMD:R_0805_2012Metric_Pad1.15x1.40mm_HandSolder" H 6700 2700 50  0001 C CNN
+F 2 "Resistor_SMD:R_0612_1632Metric_Pad1.18x3.40mm_HandSolder" H 6700 2700 50  0001 C CNN
 F 3 "" H 6700 2700 50  0001 C CNN
 	1    6700 2700
@@
 F 0 "R18" H 7650 2759 59  0000 L BNN
 F 1 "560" H 7650 2570 59  0000 L BNN
-F 2 "Resistor_SMD:R_0805_2012Metric_Pad1.15x1.40mm_HandSolder" H 7800 2700 50  0001 C CNN
+F 2 "Resistor_SMD:R_0612_1632Metric_Pad1.18x3.40mm_HandSolder" H 7800 2700 50  0001 C CNN
 F 3 "" H 7800 2700 50  0001 C CNN
 	1    7800 2700
@@
 F 0 "R2" H 5600 1500 59  0000 L BNN
 F 1 "10k" H 5550 1400 59  0000 L BNN
-F 2 "Resistor_SMD:R_0805_2012Metric_Pad1.15x1.40mm_HandSolder" H 5800 1500 50  0001 C CNN
+F 2 "Resistor_SMD:R_0612_1632Metric_Pad1.18x3.40mm_HandSolder" H 5800 1500 50  0001 C CNN
 F 3 "" H 5800 1500 50  0001 C CNN
 	1    5800 1500
@@
 Text Notes 4450 5450 2    39   ~ 0
 These resistors are chosen to get 10/3 gain
-Wire Wire Line
-	2950 3950 2950 4100
-$Comp
-L PCB_2020-rescue:GND-power #GND6
-U 1 1 6DBAC010
-P 2950 4100
-AR Path="/6DBAC010" Ref="#GND6"  Part="1"
-AR Path="/5DD5E236/6DBAC010" Ref="#GND6"  Part="1"
-AR Path="/5DF27AC1/6DBAC010" Ref="#GND06"  Part="1"
-F 0 "#GND06" H 2950 4100 50  0001 C CNN
-F 1 "GND-power" H 2850 3900 59  0000 L BNN
-F 2 "" H 2950 4100 50  0001 C CNN
-F 3 "" H 2950 4100 50  0001 C CNN
-	1    2950 4100
-	1    0    0    -1
-$EndComp
 $Comp
 L PCB_2020-rescue:R-Device R3
@@
 F 0 "R3" V 3143 3950 50  0000 C CNN
 F 1 "1000" V 3234 3950 50  0000 C CNN
-F 2 "Resistor_SMD:R_0805_2012Metric_Pad1.15x1.40mm_HandSolder" V 3280 3950 50  0001 C CNN
+F 2 "Resistor_SMD:R_0612_1632Metric_Pad1.18x3.40mm_HandSolder" V 3280 3950 50  0001 C CNN
 F 3 "" H 3350 3950 50  0001 C CNN
 	1    3350 3950
@@
 F 0 "R7" V 4093 4750 50  0000 C CNN
 F 1 "5400" V 4184 4750 50  0000 C CNN
-F 2 "Resistor_SMD:R_0805_2012Metric_Pad1.15x1.40mm_HandSolder" V 4230 4750 50  0001 C CNN
+F 2 "Resistor_SMD:R_0612_1632Metric_Pad1.18x3.40mm_HandSolder" V 4230 4750 50  0001 C CNN
 F 3 "" H 4300 4750 50  0001 C CNN
 	1    4300 4750
@@
 F 0 "R6" H 3420 3096 50  0000 L CNN
 F 1 "5400" H 3420 3005 50  0000 L CNN
-F 2 "Resistor_SMD:R_0805_2012Metric_Pad1.15x1.40mm_HandSolder" V 3280 3050 50  0001 C CNN
+F 2 "Resistor_SMD:R_0612_1632Metric_Pad1.18x3.40mm_HandSolder" V 3280 3050 50  0001 C CNN
 F 3 "" H 3350 3050 50  0001 C CNN
 	1    3350 3050
@@
 F 0 "R4" V 2893 3400 50  0000 C CNN
 F 1 "1000" V 2984 3400 50  0000 C CNN
-F 2 "Resistor_SMD:R_0805_2012Metric_Pad1.15x1.40mm_HandSolder" V 3030 3400 50  0001 C CNN
+F 2 "Resistor_SMD:R_0612_1632Metric_Pad1.18x3.40mm_HandSolder" V 3030 3400 50  0001 C CNN
 F 3 "" H 3100 3400 50  0001 C CNN
 	1    3100 3400
@@
 Wire Wire Line
 	5000 3850 5000 4750
+$Comp
+L PCB_2020:DRV8874 U3
+U 1 1 5F8C5C8E
+P 7400 6250
+F 0 "U3" H 7425 6915 50  0000 C CNN
+F 1 "DRV8874" H 7425 6824 50  0000 C CNN
+F 2 "Drivetrain_control:DRV8874PWPR" H 7400 6100 50  0001 C CNN
+F 3 "" H 7400 6100 50  0001 C CNN
+	1    7400 6250
+	1    0    0    -1
+$EndComp
+$Comp
+L PCB_2020-rescue:+12V-power #P+?
+U 1 1 5F8C884E
+P 9450 6400
+AR Path="/5F8C884E" Ref="#P+?"  Part="1"
+AR Path="/5DD5E236/5F8C884E" Ref="#P+?"  Part="1"
+AR Path="/5DF27AC1/5F8C884E" Ref="#P+0102"  Part="1"
+F 0 "#P+0102" H 9450 6400 50  0001 C CNN
+F 1 "+12V-power" H 9350 6550 59  0000 L BNN
+F 2 "" H 9450 6400 50  0001 C CNN
+F 3 "" H 9450 6400 50  0001 C CNN
+	1    9450 6400
+	1    0    0    -1
+$EndComp
+$Comp
+L PCB_2020-rescue:GND-power #PWR0103
+U 1 1 5F8C6D64
+P 6200 6500
+F 0 "#PWR0103" H 6200 6250 50  0001 C CNN
+F 1 "GND-power" H 6205 6327 50  0000 C CNN
+F 2 "" H 6200 6500 50  0001 C CNN
+F 3 "" H 6200 6500 50  0001 C CNN
+	1    6200 6500
+	1    0    0    -1
+$EndComp
+$Comp
+L PCB_2020-rescue:GND-power #PWR0105
+U 1 1 5F8D4125
+P 3350 2800
+F 0 "#PWR0105" H 3350 2550 50  0001 C CNN
+F 1 "GND-power" H 3355 2627 50  0000 C CNN
+F 2 "" H 3350 2800 50  0001 C CNN
+F 3 "" H 3350 2800 50  0001 C CNN
+	1    3350 2800
+	-1   0    0    1
+$EndComp
+Wire Wire Line
+	3350 2800 3350 2900
+$Comp
+L PCB_2020-rescue:+3V3-power #+3V?
+U 1 1 5F8E5553
+P 8550 5900
+AR Path="/5F8E5553" Ref="#+3V?"  Part="1"
+AR Path="/5DD5E236/5F8E5553" Ref="#+3V?"  Part="1"
+AR Path="/5DF27AC1/5F8E5553" Ref="#+3V0101"  Part="1"
+F 0 "#+3V0101" H 8550 5900 50  0001 C CNN
+F 1 "+3V3-power" H 8400 6050 59  0000 L BNN
+F 2 "" H 8550 5900 50  0001 C CNN
+F 3 "" H 8550 5900 50  0001 C CNN
+	1    8550 5900
+	1    0    0    -1
+$EndComp
+NoConn ~ 6800 6200
+$Comp
+L PCB_2020-rescue:+3V3-power #+3V?
+U 1 1 5F8F3B6C
+P 5800 6100
+AR Path="/5F8F3B6C" Ref="#+3V?"  Part="1"
+AR Path="/5DD5E236/5F8F3B6C" Ref="#+3V?"  Part="1"
+AR Path="/5DF27AC1/5F8F3B6C" Ref="#+3V0102"  Part="1"
+F 0 "#+3V0102" H 5800 6100 50  0001 C CNN
+F 1 "+3V3-power" H 5650 6250 59  0000 L BNN
+F 2 "" H 5800 6100 50  0001 C CNN
+F 3 "" H 5800 6100 50  0001 C CNN
+	1    5800 6100
+	1    0    0    -1
+$EndComp
+$Comp
+L PCB_2020-rescue:C-Device C1
+U 1 1 5F8F6CA9
+P 8350 6100
+F 0 "C1" V 8098 6100 50  0000 C CNN
+F 1 "0.022uF" V 8189 6100 50  0000 C CNN
+F 2 "Capacitor_SMD:C_0805_2012Metric_Pad1.18x1.45mm_HandSolder" H 8388 5950 50  0001 C CNN
+F 3 "" H 8350 6100 50  0001 C CNN
+	1    8350 6100
+	0    1    1    0
+$EndComp
+Wire Wire Line
+	8050 6100 8200 6100
+Wire Wire Line
+	8500 6100 8500 6200
+Wire Wire Line
+	8500 6200 8050 6200
+Wire Wire Line
+	8050 5900 8550 5900
+$Comp
+L PCB_2020-rescue:GND-power #PWR0104
+U 1 1 5F908D2F
+P 8700 6000
+F 0 "#PWR0104" H 8700 5750 50  0001 C CNN
+F 1 "GND-power" H 8705 5827 50  0000 C CNN
+F 2 "" H 8700 6000 50  0001 C CNN
+F 3 "" H 8700 6000 50  0001 C CNN
+	1    8700 6000
+	1    0    0    -1
+$EndComp
+Wire Wire Line
+	8050 6000 8700 6000
+Text Label 6800 6600 2    39   ~ 0
+Brake_Out_1
+Text Label 8050 6500 0    39   ~ 0
+Brake_Out_2
+$Comp
+L PCB_2020-rescue:GND-power #PWR0106
+U 1 1 5F913C37
+P 8200 6600
+F 0 "#PWR0106" H 8200 6350 50  0001 C CNN
+F 1 "GND-power" H 8205 6427 50  0000 C CNN
+F 2 "" H 8200 6600 50  0001 C CNN
+F 3 "" H 8200 6600 50  0001 C CNN
+	1    8200 6600
+	1    0    0    -1
+$EndComp
+Wire Wire Line
+	8050 6600 8200 6600
+Wire Wire Line
+	8050 6400 9250 6400
+$Comp
+L PCB_2020-rescue:C-Device C3
+U 1 1 5F91AB54
+P 9100 6300
+F 0 "C3" V 8848 6300 50  0000 C CNN
+F 1 "0.022uF" V 8939 6300 50  0000 C CNN
+F 2 "Capacitor_SMD:C_0805_2012Metric_Pad1.18x1.45mm_HandSolder" H 9138 6150 50  0001 C CNN
+F 3 "" H 9100 6300 50  0001 C CNN
+	1    9100 6300
+	0    1    1    0
+$EndComp
+Wire Wire Line
+	8050 6300 8950 6300
+Wire Wire Line
+	9250 6300 9250 6400
+Connection ~ 9250 6400
+Wire Wire Line
+	9250 6400 9450 6400
+Wire Wire Line
+	6200 6500 6550 6500
+Text GLabel 6800 5900 0    39   Input ~ 0
+Brake_PWM_1
+Wire Wire Line
+	5800 6100 6650 6100
+Text GLabel 6800 6000 0    39   Input ~ 0
+Brake_PWM_2
+Wire Wire Line
+	6650 6100 6650 6300
+Wire Wire Line
+	6650 6300 6800 6300
+Connection ~ 6650 6100
+Wire Wire Line
+	6650 6100 6800 6100
+Wire Wire Line
+	6800 6400 6550 6400
+Wire Wire Line
+	6550 6400 6550 6500
+Connection ~ 6550 6500
+Wire Wire Line
+	6550 6500 6800 6500
+$Comp
+L PCB_2020-rescue:R-Device R9
+U 1 1 5F93027B
+P 2950 4100
+F 0 "R9" V 2743 4100 50  0000 C CNN
+F 1 "1000" V 2834 4100 50  0000 C CNN
+F 2 "Resistor_SMD:R_0612_1632Metric_Pad1.18x3.40mm_HandSolder" V 2880 4100 50  0001 C CNN
+F 3 "" H 2950 4100 50  0001 C CNN
+	1    2950 4100
+	-1   0    0    1
+$EndComp
+$Comp
+L PCB_2020-rescue:R-Device R8
+U 1 1 5F930BFF
+P 2800 3950
+F 0 "R8" V 2593 3950 50  0000 C CNN
+F 1 "5000" V 2684 3950 50  0000 C CNN
+F 2 "Resistor_SMD:R_0612_1632Metric_Pad1.18x3.40mm_HandSolder" V 2730 3950 50  0001 C CNN
+F 3 "" H 2800 3950 50  0001 C CNN
+	1    2800 3950
+	0    1    1    0
+$EndComp
+Connection ~ 2950 3950
+$Comp
+L PCB_2020-rescue:GND-power #PWR0107
+U 1 1 5F93212A
+P 2950 4250
+F 0 "#PWR0107" H 2950 4000 50  0001 C CNN
+F 1 "GND-power" H 2955 4077 50  0000 C CNN
+F 2 "" H 2950 4250 50  0001 C CNN
+F 3 "" H 2950 4250 50  0001 C CNN
+	1    2950 4250
+	1    0    0    -1
+$EndComp
+$Comp
+L PCB_2020-rescue:+3V3-power #+3V?
+U 1 1 5F932831
+P 2150 3950
+AR Path="/5F932831" Ref="#+3V?"  Part="1"
+AR Path="/5DD5E236/5F932831" Ref="#+3V?"  Part="1"
+AR Path="/5DF27AC1/5F932831" Ref="#+3V0103"  Part="1"
+F 0 "#+3V0103" H 2150 3950 50  0001 C CNN
+F 1 "+3V3-power" H 2050 4100 59  0000 L BNN
+F 2 "" H 2150 3950 50  0001 C CNN
+F 3 "" H 2150 3950 50  0001 C CNN
+	1    2150 3950
+	1    0    0    -1
+$EndComp
+Wire Wire Line
+	2150 3950 2650 3950
 $EndSCHEMATC

Commit message: Updating PCB with LoRa
Parts:
- C1: value 0.022uF -> 0.022 uF; footprint Capacitor_SMD:C_0805_2012Metric_Pad1.18x1.45mm_HandSolder -> Capacitor_THT:C_Disc_D3.0mm_W1.6mm_P2.50mm
- C3: footprint Capacitor_SMD:C_0805_2012Metric_Pad1.18x1.45mm_HandSolder -> Capacitor_THT:C_Disc_D3.0mm_W1.6mm_P2.50mm
- R1, R18, R2, R3, R4, R5, R6, R7, R8, R9: footprint Resistor_SMD:R_0612_1632Metric_Pad1.18x3.40mm_HandSolder -> Resistor_THT:R_Axial_DIN0204_L3.6mm_D1.6mm_P1.90mm_Vertical
Changed lines of the file:
@@
 F 0 "R1" H 4600 1550 59  0000 L BNN
 F 1 "10k" H 4550 1450 59  0000 L BNN
-F 2 "Resistor_SMD:R_0612_1632Metric_Pad1.18x3.40mm_HandSolder" H 4800 1500 50  0001 C CNN
+F 2 "Resistor_THT:R_Axial_DIN0204_L3.6mm_D1.6mm_P1.90mm_Vertical" H 4800 1500 50  0001 C CNN
 F 3 "" H 4800 1500 50  0001 C CNN
 	1    4800 1500
@@
 F 0 "R5" H 6550 2759 59  0000 L BNN
 F 1 "560" H 6550 2570 59  0000 L BNN
-F 2 "Resistor_SMD:R_0612_1632Metric_Pad1.18x3.40mm_HandSolder" H 6700 2700 50  0001 C CNN
+F 2 "Resistor_THT:R_Axial_DIN0204_L3.6mm_D1.6mm_P1.90mm_Vertical" H 6700 2700 50  0001 C CNN
 F 3 "" H 6700 2700 50  0001 C CNN
 	1    6700 2700
@@
 AR Path="/1A44BE4A" Ref="R18"  Part="1"
 AR Path="/5DD5E236/1A44BE4A" Ref="R18"  Part="1"
-AR Path="/5DF27AC1/1A44BE4A" Ref="R18"  Part="1"
-F 0 "R18" H 7650 2759 59  0000 L BNN
+AR Path="/5DF27AC1/1A44BE4A" Ref="R10"  Part="1"
+F 0 "R10" H 7650 2759 59  0000 L BNN
 F 1 "560" H 7650 2570 59  0000 L BNN
-F 2 "Resistor_SMD:R_0612_1632Metric_Pad1.18x3.40mm_HandSolder" H 7800 2700 50  0001 C CNN
+F 2 "Resistor_THT:R_Axial_DIN0204_L3.6mm_D1.6mm_P1.90mm_Vertical" H 7800 2700 50  0001 C CNN
 F 3 "" H 7800 2700 50  0001 C CNN
 	1    7800 2700
@@
 F 0 "R2" H 5600 1500 59  0000 L BNN
 F 1 "10k" H 5550 1400 59  0000 L BNN
-F 2 "Resistor_SMD:R_0612_1632Metric_Pad1.18x3.40mm_HandSolder" H 5800 1500 50  0001 C CNN
+F 2 "Resistor_THT:R_Axial_DIN0204_L3.6mm_D1.6mm_P1.90mm_Vertical" H 5800 1500 50  0001 C CNN
 F 3 "" H 5800 1500 50  0001 C CNN
 	1    5800 1500
@@
 F 0 "R3" V 3143 3950 50  0000 C CNN
 F 1 "1000" V 3234 3950 50  0000 C CNN
-F 2 "Resistor_SMD:R_0612_1632Metric_Pad1.18x3.40mm_HandSolder" V 3280 3950 50  0001 C CNN
+F 2 "Resistor_THT:R_Axial_DIN0204_L3.6mm_D1.6mm_P1.90mm_Vertical" V 3280 3950 50  0001 C CNN
 F 3 "" H 3350 3950 50  0001 C CNN
 	1    3350 3950
@@
 F 0 "R7" V 4093 4750 50  0000 C CNN
 F 1 "5400" V 4184 4750 50  0000 C CNN
-F 2 "Resistor_SMD:R_0612_1632Metric_Pad1.18x3.40mm_HandSolder" V 4230 4750 50  0001 C CNN
+F 2 "Resistor_THT:R_Axial_DIN0204_L3.6mm_D1.6mm_P1.90mm_Vertical" V 4230 4750 50  0001 C CNN
 F 3 "" H 4300 4750 50  0001 C CNN
 	1    4300 4750
@@
 F 0 "R6" H 3420 3096 50  0000 L CNN
 F 1 "5400" H 3420 3005 50  0000 L CNN
-F 2 "Resistor_SMD:R_0612_1632Metric_Pad1.18x3.40mm_HandSolder" V 3280 3050 50  0001 C CNN
+F 2 "Resistor_THT:R_Axial_DIN0204_L3.6mm_D1.6mm_P1.90mm_Vertical" V 3280 3050 50  0001 C CNN
 F 3 "" H 3350 3050 50  0001 C CNN
 	1    3350 3050
@@
 F 0 "R4" V 2893 3400 50  0000 C CNN
 F 1 "1000" V 2984 3400 50  0000 C CNN
-F 2 "Resistor_SMD:R_0612_1632Metric_Pad1.18x3.40mm_HandSolder" V 3030 3400 50  0001 C CNN
+F 2 "Resistor_THT:R_Axial_DIN0204_L3.6mm_D1.6mm_P1.90mm_Vertical" V 3030 3400 50  0001 C CNN
 F 3 "" H 3100 3400 50  0001 C CNN
 	1    3100 3400
@@
 	1    0    0    -1
 $EndComp
-$Comp
-L PCB_2020-rescue:C-Device C1
-U 1 1 5F8F6CA9
-P 8350 6100
-F 0 "C1" V 8098 6100 50  0000 C CNN
-F 1 "0.022uF" V 8189 6100 50  0000 C CNN
-F 2 "Capacitor_SMD:C_0805_2012Metric_Pad1.18x1.45mm_HandSolder" H 8388 5950 50  0001 C CNN
-F 3 "" H 8350 6100 50  0001 C CNN
-	1    8350 6100
-	0    1    1    0
-$EndComp
 Wire Wire Line
 	8050 6100 8200 6100
@@
 F 0 "C3" V 8848 6300 50  0000 C CNN
 F 1 "0.022uF" V 8939 6300 50  0000 C CNN
-F 2 "Capacitor_SMD:C_0805_2012Metric_Pad1.18x1.45mm_HandSolder" H 9138 6150 50  0001 C CNN
+F 2 "Capacitor_THT:C_Disc_D3.0mm_W1.6mm_P2.50mm" H 9138 6150 50  0001 C CNN
 F 3 "" H 9100 6300 50  0001 C CNN
 	1    9100 6300
@@
 F 0 "R9" V 2743 4100 50  0000 C CNN
 F 1 "1000" V 2834 4100 50  0000 C CNN
-F 2 "Resistor_SMD:R_0612_1632Metric_Pad1.18x3.40mm_HandSolder" V 2880 4100 50  0001 C CNN
+F 2 "Resistor_THT:R_Axial_DIN0204_L3.6mm_D1.6mm_P1.90mm_Vertical" V 2880 4100 50  0001 C CNN
 F 3 "" H 2950 4100 50  0001 C CNN
 	1    2950 4100
@@
 F 0 "R8" V 2593 3950 50  0000 C CNN
 F 1 "5000" V 2684 3950 50  0000 C CNN
-F 2 "Resistor_SMD:R_0612_1632Metric_Pad1.18x3.40mm_HandSolder" V 2730 3950 50  0001 C CNN
+F 2 "Resistor_THT:R_Axial_DIN0204_L3.6mm_D1.6mm_P1.90mm_Vertical" V 2730 3950 50  0001 C CNN
 F 3 "" H 2800 3950 50  0001 C CNN
 	1    2800 3950
@@
 	1    0    0    -1
 $EndComp
+$Comp
+L PCB_2020-rescue:C-Device C1
+U 1 1 5FB532D1
+P 8350 6100
+F 0 "C1" V 8098 6100 50  0000 C CNN
+F 1 "0.022 uF" V 8189 6100 50  0000 C CNN
+F 2 "Capacitor_THT:C_Disc_D3.0mm_W1.6mm_P2.50mm" H 8388 5950 50  0001 C CNN
+F 3 "" H 8350 6100 50  0001 C CNN
+	1    8350 6100
+	0    1    1    0
+$EndComp
 $EndSCHEMATC

Commit message: Added AND gate for Feather LoRa, and changed over to through hole components
Parts:
- removed U3: DRV8874, Drivetrain_control:DRV8874PWPR, symbol PCB_2020:DRV8874
- added C4: 10u, Capacitor_THT:C_Disc_D3.0mm_W1.6mm_P2.50mm, symbol PCB_2020-rescue:C-Device
- added R11: R-Device, Resistor_THT:R_Axial_DIN0204_L3.6mm_D1.6mm_P1.90mm_Vertical, symbol PCB_2020-rescue:R-Device
- added R12: 4k, Resistor_THT:R_Axial_DIN0204_L3.6mm_D1.6mm_P1.90mm_Vertical, symbol PCB_2020-rescue:R-Device
- added R13: 1k, Resistor_THT:R_Axial_DIN0204_L3.6mm_D1.6mm_P1.90mm_Vertical, symbol PCB_2020-rescue:R-Device
- added U5: STK681-332-E, Drivetrain_control:STK681-332-E, symbol 2020-12-20_21-08-33:STK681-332-E
- C1: value 0.022 uF -> 47u
- C3: value 0.022uF -> 0.1u
Connections:
- net labels added: BrakeEnable
- wire segments 89 -> 106
